File: CircuitDiagram_1.0/Test_one.kicad_sch (KiCad schematic)
At the start: 27 parts, among them M1_R_1_O_2_Y_3_P_4_B_5 Stepper_Motor_unipolar_5pin, Q1 TIP122, Q2 TIP122, Q3 TIP122, Q4 TIP122, U1 4017, U2 7432

Commit message: --Added Title and dates to circuit schema --
Other:
- title: (none) -> Electromechanical Stopwatch
Changed lines of the file:
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@@
 	(generator_version "8.0")
 	(paper "A4")
+	(title_block
+		(title "Electromechanical Stopwatch")
+		(date "2024-05-20")
+	)
 	(junction
 		(at 203.2 147.32)
